Commit message: Teleop Control enabled

File: description/colours.xacro (robot description, xacro)
@@ -13,3 +13,6 @@
         <color rgba="0 0 0 1"/>
     </material>
+    <material name="red">
+        <color rgba="1 0.0 0.0 1.0"/>
+    </material>
 </robot>

File: description/robot.urdf.xacro (robot description, xacro)
@@ -3,3 +3,5 @@
     <xacro:include filename="robot_core.xacro" />
     <xacro:include filename="colours.xacro" />
+    <xacro:include filename="gazebo_control.xacro"/>
+    <xacro:include filename="lidar.xacro"/>
 </robot>

File: description/robot_core.xacro (robot description, xacro)
@@ -63,5 +63,5 @@
     </gazebo>
     <!-- RIGHT WHEEL  -->
-    <joint name="right_wheel_join" type="continuous">
+    <joint name="right_wheel_joint" type="continuous">
         <parent link="chassis"/>
         <child link="right_wheel"/>
